File: Power subsystem.kicad_sch (KiCad schematic)
At the start: 11 parts, among them J1 Conn_01x02_Pin, J2 Conn_01x04_Pin, P1 USB_C_Plug, U1 INA219AxD, U3 TP4056-42-ESOP8

Commit message: Add files via upload
Parts:
- added BT2: Battery, symbol Device:Battery
- added C3: 0.1uF, symbol Device:C
- added C4: 10uF, symbol Device:C
- added Charging, FullyCharged: LED, symbol Device:LED
- added Rch, Rf: 220, symbol Device:R
- added Rset: 1.2k, symbol Device:R
Connections:
- net GND: now also Charging.1 (K), FullyCharged.1 (K), Rset.2
- net at U3.2 (PROG): now also Rset.1
- net at U3.3 (GND): now also P1.A1 (GND), P1.A12 (GND), P1.B1 (GND), P1.B12 (GND), BT2.2 (-), C3.2, C4.2
- net at U3.4 (V_{CC}): now also P1.A4 (VBUS), P1.A9 (VBUS), P1.B4 (VBUS), P1.B9 (VBUS), U3.8 (CE), BT2.1 (+), C3.1, C4.1
- net at U3.6 (~{STDBY}): now also Rf.1
- net at U3.7 (~{CHRG}): now also Rch.1
- new net: Charging.2 (A), Rch.2
- new net: FullyCharged.2 (A), Rf.2
Other:
- moved on the sheet: U3

Commit message: Add files via upload
Connections:
- net GND: now also J2.2 (Pin_2)
- net BAT+: now reaches J1.1 (Pin_1)
- net BAT-: now reaches J1.2 (Pin_2)
- net 3V3: now reaches J2.1 (Pin_1)
- net SDA: now reaches J2.3 (Pin_3)
- net SCL: now reaches J2.4 (Pin_4)
Other:
- moved on the sheet: C1, C2, J1, J2
Changed lines of the file:
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@@
+	(wire
+		(pts
+			(xy 53.34 52.07) (xy 53.34 58.42)
+		)
+		(stroke
+			(width 0)
+			(type default)
+		)
+	)
 	(wire
 		(pts
@@
 	(wire
 		(pts
+			(xy 34.29 43.18) (xy 34.29 58.42)
+		)
+		(stroke
+			(width 0)
+			(type default)
+		)
+	)
+	(wire
+		(pts
 			(xy 115.57 68.58) (xy 115.57 73.66)
 		)
@@
 	(wire
 		(pts
+			(xy 41.91 43.18) (xy 41.91 58.42)
+		)
+		(stroke
+			(width 0)
+			(type default)
+		)
+	)
+	(wire
+		(pts
 			(xy 208.28 100.33) (xy 208.28 101.6)
 		)
@@
 	(wire
 		(pts
+			(xy 39.37 43.18) (xy 39.37 58.42)
+		)
+		(stroke
+			(width 0)
+			(type default)
+		)
+	)
+	(wire
+		(pts
 			(xy 208.28 68.58) (xy 208.28 57.15)
 		)
@@
 	(wire
 		(pts
+			(xy 50.8 52.07) (xy 50.8 58.42)
+		)
+		(stroke
+			(width 0)
+			(type default)
+		)
+	)
+	(wire
+		(pts
 			(xy 87.63 63.5) (xy 87.63 68.58)
 		)
@@
 		(pts
 			(xy 208.28 101.6) (xy 217.17 101.6)
+		)
+		(stroke
+			(width 0)
+			(type default)
+		)
+	)
+	(wire
+		(pts
+			(xy 36.83 43.18) (xy 36.83 58.42)
 		)
 		(stroke
@@
 		)
 	)
+	(label "BAT+"
+		(at 50.8 52.07 180)
+		(effects
+			(font
+				(size 1.27 1.27)
+			)
+			(justify right bottom)
+		)
+	)
+	(label "BAT-"
+		(at 53.34 52.07 0)
+		(effects
+			(font
+				(size 1.27 1.27)
+			)
+			(justify left bottom)
+		)
+	)
+	(label "GND"
+		(at 36.83 43.18 90)
+		(effects
+			(font
+				(size 1.27 1.27)
+			)
+			(justify left bottom)
+		)
+	)
+	(label "SCL"
+		(at 41.91 43.18 90)
+		(effects
+			(font
+				(size 1.27 1.27)
+			)
+			(justify left bottom)
+		)
+	)
 	(label "5v,3v3 supply"
 		(at 87.63 64.77 0)
+		(effects
+			(font
+				(size 1.27 1.27)
+			)
+			(justify left bottom)
+		)
+	)
+	(label "3V3"
+		(at 34.29 43.18 180)
+		(effects
+			(font
+				(size 1.27 1.27)
+			)
+			(justify right bottom)
+		)
+	)
+	(label "SDA"
+		(at 39.37 43.18 90)
 		(effects
 			(font
@@
 	(symbol
 		(lib_id "Device:C")
-		(at 45.72 50.8 0)
+		(at 33.02 87.63 0)
 		(unit 1)
 		(exclude_from_sim no)
@@
 		(fields_autoplaced yes)
 		(property "Reference" "C2"
-			(at 49.53 49.5299 0)
+			(at 36.83 86.3599 0)
 			(effects
 				(font
@@
 		)
 		(property "Value" "10uF"
-			(at 49.53 52.0699 0)
+			(at 36.83 88.8999 0)
 			(effects
 				(font
@@
 		)
 		(property "Footprint" ""
-			(at 46.6852 54.61 0)
+			(at 33.9852 91.44 0)
 			(effects
 				(font
@@
 		)
 		(property "Datasheet" "~"
-			(at 45.72 50.8 0)
+			(at 33.02 87.63 0)
 			(effects
 				(font
@@
 		)
 		(property "Description" "Unpolarized capacitor"
-			(at 45.72 50.8 0)
+			(at 33.02 87.63 0)
 			(effects
 				(font
@@
 	(symbol
 		(lib_id "Connector:Conn_01x02_Pin")
-		(at 73.66 52.07 0)
+		(at 50.8 63.5 90)
 		(unit 1)
 		(exclude_from_sim no)
@@
 		(fields_autoplaced yes)
 		(property "Reference" "J1"
-			(at 74.295 46.99 0)
-			(effects
-				(font
-					(size 1.27 1.27)
-				)
+			(at 54.61 61.5949 90)
+			(effects
+				(font
+					(size 1.27 1.27)
+				)
+				(justify right)
 			)
 		)
 		(property "Value" "Conn_01x02_Pin"
-			(at 74.295 49.53 0)
-			(effects
-				(font
-					(size 1.27 1.27)
-				)
+			(at 54.61 64.1349 90)
+			(effects
+				(font
+					(size 1.27 1.27)
+				)
+				(justify right)
 			)
 		)
 		(property "Footprint" ""
-			(at 73.66 52.07 0)
+			(at 50.8 63.5 0)
 			(effects
 				(font
@@
 		)
 		(property "Datasheet" "~"
-			(at 73.66 52.07 0)
+			(at 50.8 63.5 0)
 			(effects
 				(font
@@
 		)
 		(property "Description" "Generic connector, single row, 01x02, script generated"
-			(at 73.66 52.07 0)
+			(at 50.8 63.5 0)
 			(effects
 				(font
@@
 	(symbol
 		(lib_id "Connector:Conn_01x04_Pin")
-		(at 62.23 54.61 90)
+		(at 36.83 63.5 90)
 		(unit 1)
 		(exclude_from_sim no)
@@
 		(dnp no)
 		(property "Reference" "J2"
-			(at 54.61 53.975 0)
+			(at 29.21 62.865 0)
 			(effects
 				(font
@@
 		)
 		(property "Value" "Conn_01x04_Pin"
-			(at 57.15 53.975 0)
+			(at 31.75 62.865 0)
 			(effects
 				(font
@@
 		)
 		(property "Footprint" ""
-			(at 62.23 54.61 0)
+			(at 36.83 63.5 0)
 			(effects
 				(font
@@
 		)
 		(property "Datasheet" "~"
-			(at 62.23 54.61 0)
+			(at 36.83 63.5 0)
 			(effects
 				(font
@@
 		)
 		(property "Description" "Generic connector, single row, 01x04, script generated"
-			(at 62.23 54.61 0)
+			(at 36.83 63.5 0)
 			(effects
 				(font
@@
 	(symbol
 		(lib_id "Device:C")
-		(at 34.29 52.07 0)
+		(at 21.59 88.9 0)
 		(unit 1)
 		(exclude_from_sim no)
@@
 		(fields_autoplaced yes)
 		(property "Reference" "C1"
-			(at 38.1 50.7999 0)
+			(at 25.4 87.6299 0)
 			(effects
 				(font
@@
 		)
 		(property "Value" "0.1uF"
-			(at 38.1 53.3399 0)
+			(at 25.4 90.1699 0)
 			(effects
 				(font
@@
 		)
 		(property "Footprint" ""
-			(at 35.2552 55.88 0)
+			(at 22.5552 92.71 0)
 			(effects
 				(font
@@
 		)
 		(property "Datasheet" "~"
-			(at 34.29 52.07 0)
+			(at 21.59 88.9 0)
 			(effects
 				(font
@@
 		)
 		(property "Description" "Unpolarized capacitor"
-			(at 34.29 52.07 0)
-			(effects
-				(font
+			(at 21.59 88.9 0)
+			(effects
+				(font

Commit message: Add files via upload
Parts:
- removed BT1, BT2: Battery, symbol Device:Battery
Connections:
- net 5v,3v3 supply is gone; now on net +5,+3.3 V: R3.1, R5.1, U1.1 (A1), U1.5 (VS)
- net BAT+: now also U1.8 (IN+)
- net GND: now also C1.2, C2.1
- net Charging LiPo battery: now reaches C3.2, C4.2, P1.A1 (GND), P1.A12 (GND), P1.B1 (GND), P1.B12 (GND), U3.3 (GND)
- net +5,+3.3 V: now reaches C2.2
- net +5,+3.3 V: now also C1.1
- net 3V3 renamed +3.3V
Other:
- moved on the sheet: C1, C2, J1, R3, R5, Rshunt, U1

Commit message: Add files via upload
Connections:
- net BAT- is gone; now on net GND: J1.2 (Pin_2)
- net Charging LiPo battery is gone; now on net GND: C3.2, C4.2, P1.A1 (GND), P1.A12 (GND), P1.B1 (GND), P1.B12 (GND), U3.3 (GND)
- net BAT+: now also U3.5 (BAT)
- net at C3.1, C4.1, P1.A4 (VBUS)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: no longer U3.8 (CE)

Commit message: Add files via upload
Parts:
- removed P1: USB_C_Plug, symbol Connector:USB_C_Plug
- added BT1, BT2: Battery, symbol Device:Battery
- added C5: 1uF, PCM_JLCPCB:C_0402, symbol JLCPCB-Capacitors:0402,1uF
- added J3: Connector, USB-TYPE-C-16P, PCM_JLCPCB:TYPE-C-SMD_HX-TYPE-C-16PIN, symbol JLCPCB-Extended:Connector, USB-TYPE-C-16P
- added R1: 1kΩ, PCM_JLCPCB:R_0603, symbol JLCPCB-Resistors:0603,1kΩ
- added R2: 10kΩ, PCM_JLCPCB:R_0603, symbol JLCPCB-Resistors:0603,10kΩ
- added R4: 6.8kΩ, PCM_JLCPCB:R_0603, symbol JLCPCB-Resistors:0603,6.8kΩ
- added SW1: SW_SPST, symbol Switch:SW_SPST
- added U2: CH224K, Package_SO:SSOP-10-1EP_3.9x4.9mm_P1mm_EP2.1x3.3mm, symbol Interface_USB:CH224K
- added U4: ~, ETA1038:Untitled, symbol ETA1038:ETA1038
Connections:
- net BAT+: no longer U1.8 (IN+), U3.5 (BAT)
- net GND: no longer C1.2, C2.1, C3.2, C4.2, J1.2 (Pin_2), U3.3 (GND)
- net at C3.1, C4.1, U3.4 (V_{CC}): now also U3.8 (CE), BT2.1 (+), J3.A9B4 (VBUS), J3.B9A4 (VBUS), R1.1, R2.1
- net +3.3V renamed 3V3
- net +5,+3.3 V renamed 5v,3v3 supply
- net 5v,3v3 supply: no longer C1.1, C2.2
- new net: BT2.2 (-), C3.2, C4.2, C5.2, J3.A12B1 (GND), J3.B12A1 (GND), R4.2, U2.11 (GND), U3.3 (GND)
- new net: J3.A5 (CC1), U2.7 (CC1)
- new net: J3.B5 (CC2), U2.6 (CC2)
- new net: BT1.1 (+), U1.8 (IN+)
- new net: R4.1, U2.9 (CFG1)
- new net: C5.1, R1.2, U2.1 (VDD)
- new net: R2.2, U2.8 (VBUS)
- new net BAT-: J1.2 (Pin_2)
- no-connect marks 0 -> 9
Other:
- moved on the sheet: C1, C2, C3, C4, Charging, FullyCharged, J1, R3, R5, Rch, Rf, Rset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

Commit message: Add files via upload
Parts:
- removed BT1, BT2: Battery, symbol Device:Battery
- removed C5: 1uF, PCM_JLCPCB:C_0402, symbol JLCPCB-Capacitors:0402,1uF
- removed J3: Connector, USB-TYPE-C-16P, PCM_JLCPCB:TYPE-C-SMD_HX-TYPE-C-16PIN, symbol JLCPCB-Extended:Connector, USB-TYPE-C-16P
- removed R1: 1kΩ, PCM_JLCPCB:R_0603, symbol JLCPCB-Resistors:0603,1kΩ
- removed R2: 10kΩ, PCM_JLCPCB:R_0603, symbol JLCPCB-Resistors:0603,10kΩ
- removed R4: 6.8kΩ, PCM_JLCPCB:R_0603, symbol JLCPCB-Resistors:0603,6.8kΩ
- removed SW1: SW_SPST, symbol Switch:SW_SPST
- removed U2: CH224K, Package_SO:SSOP-10-1EP_3.9x4.9mm_P1mm_EP2.1x3.3mm, symbol Interface_USB:CH224K
- removed U4: ~, ETA1038:Untitled, symbol ETA1038:ETA1038
- added P1: USB_C_Plug, symbol Connector:USB_C_Plug
Connections:
- net 5v,3v3 supply is gone; now on net +5,+3.3 V: R3.1, R5.1, U1.1 (A1), U1.5 (VS)
- net BAT+: now also U1.8 (IN+)
- net GND: now also C1.2, C2.1
- net Charging LiPo battery: now reaches C3.2, C4.2, U3.3 (GND)
- net Charging LiPo battery: now also P1.A1 (GND), P1.A12 (GND), P1.B1 (GND), P1.B12 (GND)
- net at C3.1, C4.1, U3.4 (V_{CC})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: now also P1.A4 (VBUS), P1.A9 (VBUS), P1.B4 (VBUS), P1.B9 (VBUS)
- net +5,+3.3 V: now reaches C2.2
- net +5,+3.3 V: now also C1.1
- net 3V3 renamed +3.3V
- no-connect marks 9 -> 0
Other:
- moved on the sheet: C1, C2, C3, C4, Charging, FullyCharged, J1, R3, R5, Rch, Rf, Rset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
