File: Power subsystem.kicad_sch (KiCad schematic)
At the start: 55 parts, among them J1 Conn_01x02_Pin, J2 Conn_01x04_Pin, J3 Connector, USB-TYPE-C-16P, J4 Conn_02x16_Odd_Even, Q1 AO3401A, Q2 MMBT5551 200-300, Q3 2N7002, U1 INA219AxD, U10 DRV8837, U2 CH224K, U3 ETA1038S2G, U4 MR1-110-C5N-BBAA, U5 TP4056-42-ESOP8, U6 AP63203WU, U7 DRV8837, U8 DRV8837, U9 DRV8837

Commit message: Add files via upload
Parts:
- removed J1: Conn_01x02_Pin, Connector_JST:JST_PH_B2B-PH-K_1x02_P2.00mm_Vertical, symbol Connector:Conn_01x02_Pin
- removed J2: Conn_01x04_Pin, symbol Connector:Conn_01x04_Pin
- removed R10: 1kΩ, PCM_JLCPCB:R_0603, symbol JLCPCB-Resistors:0603,1kΩ
- added Q4: AO3401A, PCM_JLCPCB:Q_SOT-23, symbol PCM_JLCPCB-Transistors:PMOS,AO3401A
- added Q5: MMBT5551 200-300, PCM_JLCPCB:Q_SOT-23, symbol PCM_JLCPCB-Transistors:NPN,MMBT5551 200-300
- added R10: 10kΩ, PCM_JLCPCB:R_0603, symbol JLCPCB-Resistors:0603,10kΩ
- added R13, R14: 470Ω, PCM_JLCPCB:R_0603, symbol PCM_JLCPCB-Resistors:0603,470Ω
Connections:
- net +5V is gone; now on net 5V Out: Q1.2 (S), R5.1
- net Charging LiPo battery is gone; now on net Battery: U5.5 (BAT)
- net 5V Out: now also Q4.2 (S), R10.1
- net EXT_LOAD1_OUT: now also R13.2
- net EXT_LOAD2_OUT: now also R14.2
- net GND: now also Q5.3 (C)
- net at Q2.1 (B): now also R13.1
- net BATTERY renamed FAST_CHARGE_CTRL 
- net Load renamed LOAD1
- new net: Q4.1 (G), Q5.2 (E), R10.2
- new net: Q5.1 (B), R14.1
- new net LOAD2: Q4.3 (D)
Other:
- moved on the sheet: C3, C4, C5, Charging1, FullyCharged1, J3, Q1, Q2, Q3, R1, R12, R15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

Commit message: Add files via upload
Connections:
- net 5v,3v3 supply is gone; now on net 3V3 Out: C2.2, C6.2, R3.2, R6.2, U1.1 (A1), U1.5 (VS)
- net LOAD2 is gone; now on net CTRL_EXT_LOAD2: Q4.3 (D)
- net Battery: no longer U1.8 (IN+)
- net LOAD1 renamed CTRL_EXT_LOAD1 
- net load renamed BAT-
- new net BAT+: U1.8 (IN+)
Other:
- moved on the sheet: C14
Changed lines of the file:
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@@
 	)
 	(junction
-		(at 74.93 105.41)
-		(diameter 0)
-		(color 0 0 0 0)
-	)
-	(junction
 		(at 72.39 105.41)
 		(diameter 0)
@@
 	)
 	(junction
+		(at 74.93 104.14)
+		(diameter 0)
+		(color 0 0 0 0)
+	)
+	(junction
 		(at 118.11 107.95)
 		(diameter 0)
@@
 	(wire
 		(pts
+			(xy 237.49 33.02) (xy 237.49 43.18)
+		)
+		(stroke
+			(width 0)
+			(type default)
+		)
+	)
+	(wire
+		(pts
 			(xy 64.77 118.11) (xy 64.77 105.41)
 		)
@@
 	(wire
 		(pts
-			(xy 87.63 102.87) (xy 87.63 105.41)
+			(xy 86.36 102.87) (xy 86.36 107.95)
 		)
 		(stroke
@@
 	(wire
 		(pts
-			(xy 74.93 105.41) (xy 74.93 107.95)
-		)
-		(stroke
-			(width 0)
-			(type default)
-		)
-	)
-	(wire
-		(pts
 			(xy 252.73 36.83) (xy 252.73 45.72)
 		)
@@
 	(wire
 		(pts
+			(xy 86.36 102.87) (xy 87.63 102.87)
+		)
+		(stroke
+			(width 0)
+			(type default)
+		)
+	)
+	(wire
+		(pts
 			(xy 78.74 153.67) (xy 78.74 158.75)
 		)
@@
 	(wire
 		(pts
+			(xy 78.74 104.14) (xy 74.93 104.14)
+		)
+		(stroke
+			(width 0)
+			(type default)
+		)
+	)
+	(wire
+		(pts
 			(xy 226.06 52.07) (xy 226.06 62.23)
 		)
@@
 	(wire
 		(pts
+			(xy 74.93 104.14) (xy 74.93 107.95)
+		)
+		(stroke
+			(width 0)
+			(type default)
+		)
+	)
+	(wire
+		(pts
 			(xy 147.32 52.07) (xy 149.86 52.07)
 		)
@@
 	(wire
 		(pts
-			(xy 73.66 67.31) (xy 73.66 62.23)
+			(xy 73.66 62.23) (xy 73.66 67.31)
 		)
 		(stroke
@@
 	(wire
 		(pts
-			(xy 74.93 105.41) (xy 80.01 105.41)
+			(xy 120.65 107.95) (xy 120.65 110.49)
 		)
 		(stroke
@@
 	(wire
 		(pts
-			(xy 120.65 107.95) (xy 120.65 110.49)
+			(xy 247.65 114.3) (xy 247.65 120.65)
 		)
 		(stroke
@@
 	(wire
 		(pts
-			(xy 247.65 114.3) (xy 247.65 120.65)
+			(xy 190.5 144.78) (xy 190.5 125.73)
 		)
 		(stroke
@@
 	(wire
 		(pts
-			(xy 190.5 144.78) (xy 190.5 125.73)
+			(xy 78.74 107.95) (xy 78.74 104.14)
 		)
 		(stroke
@@
 	(wire
 		(pts
-			(xy 74.93 97.79) (xy 74.93 105.41)
+			(xy 74.93 97.79) (xy 74.93 104.14)
 		)
 		(stroke
@@
 	(wire
 		(pts
-			(xy 237.49 33.02) (xy 237.49 40.64)
-		)
-		(stroke
-			(width 0)
-			(type default)
-		)
-	)
-	(wire
-		(pts
 			(xy 274.32 151.13) (xy 274.32 152.4)
 		)
@@
 		)
 	)
+	(label "CTRL_EXT_LOAD1 "
+		(at 237.49 43.18 0)
+		(effects
+			(font
+				(size 1.27 1.27)
+			)
+			(justify left bottom)
+		)
+	)
 	(label "MOTOR4_CTRL2"
 		(at 119.38 176.53 180)
@@
 		)
 	)
-	(label "load"
+	(label "BAT-"
 		(at 86.36 16.51 180)
 		(effects
@@
 		)
 	)
-	(label "LOAD2"
-		(at 240.03 76.2 0)
+	(label "CTRL_EXT_LOAD2"
+		(at 240.03 76.2 180)
 		(effects
 			(font
 				(size 1.27 1.27)
 			)
-			(justify left bottom)
+			(justify right bottom)
 		)
 	)
@@
 		)
 	)
+	(label "3V3 Out"
+		(at 73.66 67.31 0)
+		(effects
+			(font
+				(size 1.27 1.27)
+			)
+			(justify left bottom)
+		)
+	)
 	(label "Motor4_B_OUT"
 		(at 33.02 143.51 180)
@@
 		)
 	)
-	(label "Battery"
+	(label "BAT+"
 		(at 92.71 43.18 0)
 		(effects
@@
 		)
 	)
-	(label "5v,3v3 supply"
-		(at 73.66 66.04 180)
-		(effects
-			(font
-				(size 1.27 1.27)
-			)
-			(justify right bottom)
-		)
-	)
 	(label "MOTOR3_CTRL1"
 		(at 71.12 179.07 180)
@@
 		)
 	)
-	(label "LOAD1"
-		(at 237.49 40.64 0)
-		(effects
-			(font
-				(size 1.27 1.27)
-			)
-			(justify left bottom)
-		)
-	)
 	(label "MOTOR2_CTRL1"
 		(at 45.72 140.97 0)
@@
 	(symbol
 		(lib_id "PCM_JLCPCB-Capacitors:0603,100nF")
-		(at 83.82 105.41 90)
+		(at 82.55 107.95 90)
 		(unit 1)
 		(exclude_from_sim no)
@@
 		(on_board yes)
 		(dnp no)
-		(fields_autoplaced yes)
 		(property "Reference" "C14"
-			(at 83.82 96.52 90)
+			(at 79.756 105.156 0)
 			(effects
 				(font
@@
 		)
 		(property "Value" "100nF"
-			(at 83.82 99.06 90)
+			(at 82.296 105.664 90)
 			(effects
 				(font
@@
 		)
 		(property "Footprint" "PCM_JLCPCB:C_0603"
-			(at 83.82 107.188 90)
+			(at 82.55 109.728 90)
 			(effects
 				(font
@@
 		)
 		(property "Datasheet" "https://www.lcsc.com/datasheet/lcsc_datasheet_2211101700_YAGEO-CC0603KRX7R9BB104_C14663.pdf"
-			(at 83.82 105.41 0)
+			(at 82.55 107.95 0)
 			(effects
 				(font
@@
 		)
 		(property "Description" "50V 100nF X7R ±10% 0603 Multilayer Ceramic Capacitors MLCC - SMD/SMT ROHS"
-			(at 83.82 105.41 0)
+			(at 82.55 107.95 0)
 			(effects
 				(font
@@
 		)
 		(property "LCSC" "C14663"
-			(at 83.82 105.41 0)
+			(at 82.55 107.95 0)
 			(effects
 				(font
@@
 		)
 		(property "Stock" "56668771"
-			(at 83.82 105.41 0)
+			(at 82.55 107.95 0)
 			(effects
 				(font
@@
 		)
 		(property "Price" "0.006USD"
-			(at 83.82 105.41 0)
+			(at 82.55 107.95 0)
 			(effects
 				(font
@@
 		)
 		(property "Process" "SMT"
-			(at 83.82 105.41 0)
+			(at 82.55 107.95 0)
 			(effects
 				(font
@@
 		)
 		(property "Minimum Qty" "20"
-			(at 83.82 105.41 0)
+			(at 82.55 107.95 0)
 			(effects
 				(font
@@
 		)
 		(property "Attrition Qty" "6"
-			(at 83.82 105.41 0)
+			(at 82.55 107.95 0)
 			(effects
 				(font
@@
 		)
 		(property "Class" "Basic Component"
-			(at 83.82 105.41 0)
+			(at 82.55 107.95 0)
 			(effects
 				(font
@@
 		)
 		(property "Category" "Capacitors,Multilayer Ceramic Capacitors MLCC - SMD/SMT"
-			(at 83.82 105.41 0)
+			(at 82.55 107.95 0)
 			(effects
 				(font
@@
 		)
 		(property "Manufacturer" "YAGEO"
-			(at 83.82 105.41 0)
+			(at 82.55 107.95 0)
 			(effects
 				(font
@@
 		)
 		(property "Part" "CC0603KRX7R9BB104"
-			(at 83.82 105.41 0)
+			(at 82.55 107.95 0)
 			(effects
 				(font
@@
 		)
 		(property "Voltage Rated" "50V"
-			(at 83.82 101.6 90)
+			(at 82.55 104.14 90)
 			(effects
 				(font
@@
 		)
 		(property "Tolerance" "±10%"
-			(at 83.82 105.41 0)
+			(at 82.55 107.95 0)
 			(effects
 				(font
@@
 		)
 		(property "Capacitance" "100nF"
-			(at 83.82 105.41 0)
+			(at 82.55 107.95 0)
 			(effects
 				(font
@@
 		)
 		(property "Temperature Coefficient" "X7R"
-			(at 83.82 105.41 0)
+			(at 82.55 107.95 0)
 			(effects
 				(font

Commit message: Add files via upload
Parts:
- removed Rshunt: 0.05, symbol Device:R
- added J1: Conn_01x02_Pin, Connector_JST:JST_PH_B2B-PH-K_1x02_P2.00mm_Vertical, symbol Connector:Conn_01x02_Pin
- added R16: MS122WJ050MT4E, myparts:R2512, symbol myparts:MS122WJ050MT4E
- added TP1, TP10, TP11, TP12, TP2, TP3, TP4, TP5, TP6, TP7, TP8, TP9: TestPoint, TestPoint:TestPoint_Pad_2.0x2.0mm, symbol Connector:TestPoint
- Charging1: footprint (none) -> LED_SMD:LED_0805_2012Metric_Pad1.15x1.40mm_HandSolder
- FullyCharged1: footprint (none) -> LED_SMD:LED_1206_3216Metric_Pad1.42x1.75mm_HandSolder
Connections:
- net BAT+ is gone; now on net Battery: U1.8 (IN+)
- net 3V3 Out: now also TP2.1
- net 5V Out: now also TP5.1
- net Battery: now also U4.1, J1.1 (Pin_1), TP4.1; no longer U4.2
- net EXT_LOAD1_OUT: now also TP6.1
- net EXT_LOAD2_OUT: now also TP7.1
- net FAST_CHARGE_CTRL : now also TP11.1, TP12.1
- net GND: now also C1.1, C10.1, C12.2, C13.2, C14.2, C15.2, C16.2, C17.2, C18.2, C19.2, C20.2, C7.2, C8.2, C9.1, J3.S1 (SHIELD), R11.1, U10.4 (GND), U10.9 (GND), U3.2 (GND), U5.1 (TEMP), U6.4 (GND), U7.4 (GND), U7.9 (GND), U8.4 (GND), U8.9 (GND), U9.4 (GND), U9.9 (GND), J1.2 (Pin_2), R16.2
- net HV: now also C3.1, C4.1, J3.A9B4 (VBUS), J3.B9A4 (VBUS), R1.1, R2.1, U5.4 (V_{CC}), U5.8 (CE), TP8.1
- net I2C1_SCL: now also R6.1, U1.4 (SCL)
- net I2C1_SDA: now also R3.1, U1.3 (SDA)
- net Motor2_A_OUT: no longer J4.3 (Pin_3), U10.2 (OUT1)
- net at R7.1, U5.6 (~{STDBY}): now also TP10.1
- net at L1.1, U3.6 (SW): now also TP3.1
- net at C11.2, L2.1, U6.6 (BST): now also TP1.1
- net at R8.1, U5.7 (~{CHRG}): now also TP9.1
- net at U1.7 (IN-): now also R16.1
- net at J4.14 (Pin_14): now also U4.2; no longer U4.1
- new net Motor4_A_OUT: J4.3 (Pin_3), U10.2 (OUT1)
- no-connect marks 9 -> 11
Other:
- moved on the sheet: J4, U4
