File: Power subsystem (1).kicad_sch (KiCad schematic)
At the start: 24 parts, among them J1 Conn_01x02_Pin, J2 Conn_01x04_Pin, J3 Connector, USB-TYPE-C-16P, SW1 SW_SPST, U1 INA219AxD, U2 CH224K, U5 TP4056-42-ESOP8

Commit message: Add files via upload
Parts:
- added Q1: AO3401A, PCM_JLCPCB:Q_SOT-23, symbol PCM_JLCPCB-Transistors:PMOS,AO3401A
- added Q2: MMBT5551 200-300, PCM_JLCPCB:Q_SOT-23, symbol PCM_JLCPCB-Transistors:NPN,MMBT5551 200-300
- added R10: 1kΩ, PCM_JLCPCB:R_0603, symbol JLCPCB-Resistors:0603,1kΩ
- added R5: 10kΩ, PCM_JLCPCB:R_0603, symbol JLCPCB-Resistors:0603,10kΩ
Connections:
- net GND: now also Q2.3 (C)
- new net: Q2.1 (B), R10.2
- new net: Q1.1 (G), Q2.2 (E), R5.2
- new net +5V: Q1.2 (S), R5.1
- new net Load: Q1.3 (D)
- new net M.C output: R10.1

Commit message: Add files via upload
Parts:
- removed R9: 1.2kΩ, PCM_JLCPCB:R_0603, symbol PCM_JLCPCB-Resistors:0603,1.2kΩ
- added BT1: Battery, symbol Device:Battery
- added Q3: MMBT5401 200-300, PCM_JLCPCB:Q_SOT-23, symbol PCM_JLCPCB-Transistors:PNP,MMBT5401 200-300
- added R12: 6.2kΩ, PCM_JLCPCB:R_0603, symbol PCM_JLCPCB-Resistors:0603,6.2kΩ
- added R13: 100kΩ, PCM_JLCPCB:R_0402, symbol PCM_JLCPCB-Resistors:0402,100kΩ
- added R14: 33kΩ, PCM_JLCPCB:R_0603, symbol PCM_JLCPCB-Resistors:0603,33kΩ
- added Rlow: 2kΩ, PCM_JLCPCB:R_0603, symbol PCM_JLCPCB-Resistors:0603,2kΩ
Connections:
- net GND: now also BT1.2 (-), R14.2, Rlow.2
- net at U5.2 (PROG): now also Q3.2 (E)
- new net: BT1.1 (+), R13.1
- new net: Q3.1 (B), R13.2, R14.1
- new net: Q3.3 (C), Rlow.1
Other:
- moved on the sheet: Q2
